File: KiCad Projects/ShellDeck-KYB/ShellDeck-KYB.kicad_pcb (KiCad board)
At the start: 2 copper layers, 330 x 139.9 mm, 257 parts, among them J1 M55-6001242R, J2 M55-6001242R, SW1 1U, SW10 1U, SW11 1U, SW12 1U, SW13 1U, SW14 1U, SW15 1U, SW16 1U, SW17 1U, SW18 1U, SW19 1U, SW2 1U, SW20 1U, SW21 1U, SW22 1U, SW23 1U, SW24 1U, SW25 1U, SW26 1U, SW27 1U, SW28 1U, SW29 1U, SW3 1U, SW30 1U, SW31 1U, SW32 1U, SW33 1U, SW34 1U, SW35 1U, SW36 1U, SW37 1U, SW38 1U, SW39 1U, SW4 1U, SW40 1U, SW41 1U, SW42 1U, SW43 1U, SW44 1U, SW45 1U, SW46 1U, SW47 1U, SW48 1U, SW49 1U, SW5 1U, SW50 1U, SW51 1U, SW52 1U, SW53 1U, SW54 1U, SW6 1U, SW7 1U, SW8 1U, SW9 1U, U1 W25Q128JVSIM_TR, U100 SOT-23-5, U2 QFN-80-1EP_10x10mm_P0.4mm_EP3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, Y1 Crystal_SMD_Abracon_ABM8G-4Pi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

Commit message: added 5v to 3v power convert and internal 3v lines
Parts:
- removed C9: C_0603, Capacitor_SMD:C_0603_1608Metric
- added C10: C_0603, Capacitor_SMD:C_0603_1608Metric, B.Cu at (186.5, 95.1)
- added C16: C_0603, Capacitor_SMD:C_0603_1608Metric, B.Cu at (195.3, 71.0)
- added C16: C_0603, Capacitor_SMD:C_0603_1608Metric, B.Cu at (197.5, 71.0)
- added R6: R_0603, Resistor_SMD:R_0603_1608Metric, B.Cu at (196.4, 67.8)
- added TP: TestPoint_Pad_D3.0mm, TestPoint:TestPoint_Pad_D3.0mm, B.Cu at (186.7, 100.4)
- added TP: TestPoint_Pad_D3.0mm, TestPoint:TestPoint_Pad_D3.0mm, B.Cu at (186.7, 105.6)
- added U100: AP2112K-3.3TRG1, Package_TO_SOT_SMD:SC-74A-5_1.55x2.9mm_P0.95mm, B.Cu at (182.2, 95.0)
Routing:
- net +3V3: track 60.3 -> 120.9 mm, vias 0 -> 1
- net RESET: track 17.4 -> 22.4 mm
- net GND: track 113.3 -> 115.8 mm, vias 57 -> 58
- net (no net): vias 0 -> 2
