File: KiCad Projects/ShellDeck-RP2040/ShellDeck-RP2040.kicad_pcb (KiCad board)
At the start: 2 copper layers, 330 x 139.9 mm, 256 parts, among them J1 M55-6001242R, J2 M55-6001242R, SW1 1U, SW10 1U, SW11 1U, SW12 1U, SW13 1U, SW14 1U, SW15 1U, SW16 1U, SW17 1U, SW18 1U, SW19 1U, SW2 1U, SW20 1U, SW21 1U, SW22 1U, SW23 1U, SW24 1U, SW25 1U, SW26 1U, SW27 1U, SW28 1U, SW29 1U, SW3 1U, SW30 1U, SW31 1U, SW32 1U, SW33 1U, SW34 1U, SW35 1U, SW36 1U, SW37 1U, SW38 1U, SW39 1U, SW4 1U, SW40 1U, SW41 1U, SW42 1U, SW43 1U, SW44 1U, SW45 1U, SW46 1U, SW47 1U, SW48 1U, SW49 1U, SW5 1U, SW50 1U, SW51 1U, SW52 1U, SW53 1U, SW54 1U, SW6 1U, SW7 1U, SW8 1U, SW9 1U, U1 W25Q128JVSIM_TR, U3 QFN-56-1EP_7x7mm_P0.4mm_EP3.2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, U4 AP2112K-3.3TRG1, U5 SOT-23-5, Y1 Crystal_SMD_Abracon_ABM8G-4Pi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

Commit message: smol changes
Parts:
- removed C5: C_0603, Capacitor_SMD:C_0603_1608Metric
- removed SW51: 1U, Key_Switch_MX_LP:Gateron-KS33-Hotswap-1U
- removed the SW52 at (153.3, 175.1)
- added SW52: 2U, KiCad Libs:Gateron-KS33-Hotswap-2U, B.Cu at (261.6, 175.0)
- added SW52: 2U, KiCad Libs:Gateron-KS33-Hotswap-2U, B.Cu at (153.5, 175.0)
- moved D44 9.67 mm to (280.5, 184.7)
- moved D48 8.82 mm to (171.4, 184.7)
- moved BOOT1 3.15 mm to (226.1, 64.7)
- moved C17 3.06 mm to (212.8, 79.6), turned to 0 degrees
- moved LED52 0.17 mm to (152.8, 169.9)
- moved LED51 0.10 mm to (260.9, 169.9)
Connections:
- net BOOT renamed ~{BOOT}
- U3 pad 28: (no net) -> RGB
- U3 pad 31: (no net) -> SDA
- U3 pad 32: (no net) -> SCL
- U3 pad 34: (no net) -> OLED_CS
- U3 pad 35: (no net) -> OLED_DC
- U3 pad 36: (no net) -> OLED_RST
- U3 pad 37: (no net) -> TRACKPAD_CS
- U3 pad 38: (no net) -> SCK
- U3 pad 39: (no net) -> MOSI
- U3 pad 40: (no net) -> MISO
- U3 pad 41: (no net) -> TRACKPAD_DR
Routing:
- net (no net): track 225.3 -> 243.6 mm
- net +3V3: track 66.3 -> 71.7 mm, vias 2 -> 4
- net ~{BOOT}: track 11.8 -> 15.6 mm
- net ROW4: track 216.8 -> 214.7 mm
Other:
- outline, holes or cut-outs redrawn

Commit message: started work on the 3d models
Parts:
- C1, C10, C12, C14, C15, C16, C17, C19, C2, C3, C4, C9: value C_0603 -> 0.1uF
- C12: value C_0603 -> 15pF
- C20: value C_0603 -> 12pF
- R2, R6: value R_0603 -> 1K
- R3, R5: value R_0603 -> 10K
