File: KiCad Projects/CM5-FatherBoard/CM5-FatherBoard.kicad_sch (KiCad schematic)
At the start: 0 parts

Commit message: started and finished the hdmi ribbon to male converter
Parts:
- added J1: USB_C_Receptacle, symbol Connector:USB_C_Receptacle
- added J2: HDMI_A, symbol Connector:HDMI_A
- added U1: CM5108032, KicadLibs:MODULE_CM5108032, symbol CM5108032:CM5108032
- added U2: USB2514B_Bi, Package_DFN_QFN:QFN-36-1EP_6x6mm_P0.5mm_EP3.7x3.7mm, symbol Interface_USB:USB2514B_Bi
Connections:
- new net: U1.SH1 (MOUNTING_PADS), U1.SH2 (MOUNTING_PADS), U1.SH3 (MOUNTING_PADS), U1.SH4 (MOUNTING_PADS)
- new net: J1.A1 (GND), J1.A12 (GND), J1.B1 (GND), J1.B12 (GND)
- new net: J1.A4 (VBUS), J1.A9 (VBUS), J1.B4 (VBUS), J1.B9 (VBUS)
- new net +5V(INPUT): U1.77 (+5V(INPUT)), U1.79 (+5V(INPUT)), U1.81 (+5V(INPUT)), U1.83 (+5V(INPUT)), U1.85 (+5V(INPUT)), U1.87 (+5V(INPUT))
- new net CM5_1.8V(OUTPUT): U1.88 (CM5_1.8V(OUTPUT)), U1.90 (CM5_1.8V(OUTPUT))
- new net CM5_3.3V(OUTPUT): U1.84 (CM5_3.3V(OUTPUT)), U1.86 (CM5_3.3V(OUTPUT))
- new net GND: U1.1 (GND), U1.107 (GND), U1.108 (GND), U1.113 (GND), U1.114 (GND), U1.119 (GND), U1.120 (GND), U1.125 (GND), U1.126 (GND), U1.13 (GND), U1.131 (GND), U1.132 (GND), U1.137 (GND), U1.138 (GND), U1.14 (GND), U1.144 (GND), U1.150 (GND), U1.155 (GND), U1.156 (GND), U1.161 (GND), U1.162 (GND), U1.167 (GND), U1.168 (GND), U1.173 (GND), U1.174 (GND), U1.179 (GND), U1.180 (GND), U1.185 (GND), U1.186 (GND), U1.191 (GND), U1.192 (GND), U1.197 (GND), U1.198 (GND), U1.2 (GND), U1.22 (GND), U1.23 (GND), U1.32 (GND), U1.33 (GND), U1.42 (GND), U1.43 (GND), U1.52 (GND), U1.53 (GND), U1.59 (GND), U1.60 (GND), U1.65 (GND), U1.66 (GND), U1.7 (GND), U1.71 (GND), U1.74 (GND), U1.8 (GND), U1.98 (GND)
