File: KiCad Projects/CM5-FatherBoard/HDMI-Ribbon-to-male/HDMI-Ribbon-to-male.kicad_sch (KiCad schematic)
At the start: 2 parts

Commit message: updated schematic
Parts:
- CN1: footprint Connector_Video:HDMI_A_Contact_Technology_19APL2_Horizontal -> ProLib_pcs_2026-03-28:HDMI-SMD_HYC109-HDMIA19-160
- renumbered e to e1
Changed lines of the file:
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@@
 			)
 		)
-		(property "Footprint" "Connector_Video:HDMI_A_Contact_Technology_19APL2_Horizontal"
+		(property "Footprint" "ProLib_pcs_2026-03-28:HDMI-SMD_HYC109-HDMIA19-160"
 			(at 246.38 76.2 0)
 			(effects
@@
 		(dnp no)
 		(fields_autoplaced yes)
-		(property "Reference" "e"
+		(property "Reference" "e1"
 			(at 189.23 74.9299 0)
 			(effects
@@
 			(project "HDMI-Ribbon-to-male"
 				(path "/f1b1d8fb-1932-4d4d-8965-9f5eb9872431"
-					(reference "e")
+					(reference "e1")
 					(unit 1)
 				)
